File: Main PCB/GlowSignMainPCB.kicad_sch (KiCad schematic)
At the start: 127 parts, among them P1 RoundConnectorPadHole, P2 RoundConnectorPadHole, P3 RoundConnectorPadHole, P4 RoundConnectorPadHole, P5 RoundConnectorPadHole, P6 RoundConnectorPadHole, P7 RoundConnectorPadHole, P8 RoundConnectorPadHole, SW1 TS-1185EC-C-D-B, SW2 TS-1185EC-C-D-B, SW3 TS-1185EC-C-D-B, U1 AP40P05, U10 TP4056, U11 DW01A, U12 SMTSO3015CTJ, U13 SMTSO3015CTJ, U14 SMTSO3015CTJ, U15 SMTSO3015CTJ, U18 BL1117-33CX, U2 SS54, U20 GMA4030H11-F26, U26 M1250RS-02P, U3 SN74AHCT32QPWRQ1, U4 ESP32-WROOM-32E, U5 FP6298XR-G1, U6 SS54, U7 CP2102-GMR, U8 UMH3N, U9 FS8205A

Commit message: updated mic and levelshifter
Parts:
- removed U20: GMA4030H11-F26, footprint:MIC-SMD_8P-L3.0-W4.0-P0.85-BL, symbol MyParts:GMA4030H11-F26
- removed U3: SN74AHCT32QPWRQ1, footprint:TSSOP-14_L5.0-W4.4-P0.65-LS6.5-BL, symbol MyParts:SN74AHCT32QPWRQ1
- added C47: 10uF, Capacitor_SMD:C_0603_1608Metric_Pad1.08x0.95mm_HandSolder, symbol Device:0.1uF 0603
- added C48: 0.1uF, Capacitor_SMD:C_0603_1608Metric_Pad1.08x0.95mm_HandSolder, symbol Device:C
- added U20: MSM261D4030H1CPM, footprint:MIC-SMD_8P-L3.0-W4.0-P0.85-BL, symbol MyParts:MSM261D4030H1CPM
- added U3: (no value), symbol MyParts:SN74LVC2T45DCUR
- C10: 1500+ (none) -> €0.0119; 50+ (none) -> €0.0171; 500+ (none) -> €0.0141; LCSC Part # C14663 -> C597194; LCSC link (none) -> https://lcsc.com/product-detail/Multilayer-Ceramic-Capacito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; Manufacturer (none) -> AVX; Mfr. Part # (none) -> 06035C104K4Z2A; Package (none) -> 0603
- C11, C14: value (none) -> 10uF; footprint (none) -> Capacitor_SMD:C_0603_1608Metric_Pad1.08x0.95mm_HandSolder
- C8, C9: value 1nF -> 1uF
- R16: value 73K -> 33K
- R17: value 10K -> 5.1K
Connections:
- net +3V3: now also C2.1, C47.2, U20.1 (VDD), U3.8 (VCCB)
- net +5V: now also C48.1, U3.1 (VCCA); no longer C2.1
- net GND: now also C47.1, C48.2, U20.5 (GND), U20.6 (GND), U20.7 (GND), U20.8 (GND), U3.3 (A2), U3.4 (GND), U3.5 (DIR), U3.6 (B2)
- net IO14/SCK: now also U20.3 (CLK)
- net IO15/WS: now also U20.2 (L/R)
- net IO16/LED1: now also U3.7 (B1)
- net IO32/SD: now also U20.4 (DATA)
- net at R1.1: now also U3.2 (A1)
Other:
- moved on the sheet: C2, R1

Commit message: made improvements and started creating usb-c only version
Parts:
- removed P1, P2, P3, P4, P5, P6, P7, P8: RoundConnectorPadHole, footprint:RoundSolderPadHole, symbol MyParts:RoundConnectorPadHole
- removed U12, U13, U14, U15: SMTSO3015CTJ, footprint:SMTSO3030CTJ, symbol MyParts:SMTSO3015CTJ
- C1, C5, C7: value 10uF -> (none); footprint Capacitor_SMD:C_0603_1608Metric_Pad1.08x0.95mm_HandSolder -> (none); LCSC # (none) -> C19702; LCSC Part # C19702 -> (none)
- C10: value 0.1uF -> (none); footprint Capacitor_SMD:C_0603_1608Metric_Pad1.08x0.95mm_HandSolder -> (none); 1500+ €0.0119 -> (none); 50+ €0.0171 -> (none); 500+ €0.0141 -> (none); LCSC # (none) -> C14663; LCSC Part # C597194 -> (none); LCSC link https://lcsc.com/product-detail/Multilayer-Ceramic-Capacito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 -> (none); Manufacturer AVX -> (none); Mfr. Part # 06035C104K4Z2A -> (none); Package 0603 -> (none)
- C11, C14: value 10uF -> (none); footprint Capacitor_SMD:C_0603_1608Metric_Pad1.08x0.95mm_HandSolder -> (none)
- C12, C13, C16, C17: value 22uF -> (none); footprint Capacitor_SMD:C_0603_1608Metric_Pad1.08x0.95mm_HandSolder -> (none); LCSC # (none) -> C59461
- C15: value 0.1uF -> (none); footprint Capacitor_SMD:C_0603_1608Metric_Pad1.08x0.95mm_HandSolder -> (none); 1500+ €0.0119 -> (none); 50+ €0.0171 -> (none); 500+ €0.0141 -> (none); LCSC # (none) -> C14663; LCSC Part # C597194 -> (none); LCSC link https://lcsc.com/product-detail/Multilayer-Ceramic-Capacito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 -> (none); Manufacturer AVX -> (none); Mfr. Part #  06035C104K4Z2A -> (none); Package 0603 -> (none)
- C18, C19, C20, C21, C22, C23, C24, C25, C26, C27, C28, C29, C30, C31, C32, C33, C34, C35, C36, C37, C38, C39, C40, C41, C42, C43, C44, C45, C46: value 0.1uf -> (none); footprint Capacitor_SMD:C_0603_1608Metric_Pad1.08x0.95mm_HandSolder -> (none); LCSC # (none) -> C14663
- C2, C48: value 0.1uF -> (none); footprint Capacitor_SMD:C_0603_1608Metric_Pad1.08x0.95mm_HandSolder -> (none)
- C3: value 220uF 10V -> (none); footprint Capacitor_SMD:CP_Elec_6.3x5.4 -> (none); LCSC # (none) -> C267466; LCSC Part # C267466 -> (none)
- C4: value 4.7uF 6.3V 10% -> (none); footprint Capacitor_SMD:C_0603_1608Metric_Pad1.08x0.95mm_HandSolder -> (none)
- C47: value 10uF -> (none); footprint Capacitor_SMD:C_0603_1608Metric_Pad1.08x0.95mm_HandSolder -> (none); 1500+ €0.0119 -> (none); 50+ €0.0171 -> (none); 500+ €0.0141 -> (none); LCSC # (none) -> C19702; LCSC Part # C597194 -> (none); LCSC link https://lcsc.com/product-detail/Multilayer-Ceramic-Capacito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 -> (none); Manufacturer AVX -> (none); Mfr. Part # 06035C104K4Z2A -> (none); Package 0603 -> (none)
- C6: value 0.1uF -> (none); footprint Capacitor_SMD:C_0603_1608Metric_Pad1.08x0.95mm_HandSolder -> (none); LCSC # (none) -> C14663; LCSC Part # C14663 -> (none)
- C8, C9: value 1uF -> (none); footprint Capacitor_SMD:C_0603_1608Metric_Pad1.08x0.95mm_HandSolder -> (none); LCSC # (none) -> C15849; LCSC Part # C1588 -> (none)
- D1: value green LED -> (none); footprint LED_SMD:LED_0603_1608Metric_Pad1.05x0.95mm_HandSolder -> (none); 20+ €0.0212 -> (none); 200+ €0.0173 -> (none); LCSC # (none) -> C193901; LCSC Part # C193901 -> (none); LCSC link https://lcsc.com/product-detail/Light-Emitting-Diodes-LED_F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 -> (none); Manufacturer Foshan NationStar Optoelectronics -> (none); Mfr. Part # NCD0603C2 -> (none); Package 0603 -> (none)
- D10, D11, D12, D13, D14, D15, D16, D17, D18, D19, D20, D21, D22, D23, D24, D25, D26, D8, D9: value WS2812B -> (none); footprint LED_SMD:LED_WS2812B_PLCC4_5.0x5.0mm_P3.2mm -> (none)
- D2: value red LED -> (none); footprint LED_SMD:LED_0603_1608Metric_Pad1.05x0.95mm_HandSolder -> (none); 50+ €0.0166 -> (none); 500+ €0.0141 -> (none); LCSC # (none) -> C72044; LCSC Part # C72044 -> (none); LCSC link https://lcsc.com/product-detail/Light-Emitting-Diodes-LED_E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 -> (none); Manufacturer Everlight Elec -> (none); Mfr. Part # 19-217/R6C-AL1M2VY/3T -> (none); Package 0603 -> (none)
- D27, D28, D29, D3, D30, D31, D4, D5, D6, D7: value WS2812B-4020 -> (none); footprint footprint:LED-SMD_WS2812B-4020 -> (none)
- F1, F2: value BSMD1812-300-16V -> (none); footprint Fuse:Fuse_1812_4532Metric_Pad1.30x3.40mm_HandSolder -> (none)
- L1: value CKCS5040-3_3UH_M -> (none); footprint footprint:IND-SMD_L5.0-W5.0 -> (none)
- R1: value 62 -> (none); footprint Resistor_SMD:R_0603_1608Metric_Pad0.98x0.95mm_HandSolder -> (none)
- R10, R11, R13: value 1K -> (none); footprint Resistor_SMD:R_0603_1608Metric_Pad0.98x0.95mm_HandSolder -> (none); 100+ €0.0012 -> (none); 1000+ €0.001 -> (none); LCSC # (none) -> C21190; LCSC Part # C115325 -> (none); LCSC link https://lcsc.com/product-detail/Chip-Resistor-Surface-Mount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 -> (none); Manufacturer FH(Guangdong Fenghua Advanced Tech) -> (none); Mfr. Part # RS-03K1001FT -> (none); Package 0603 -> (none)
- R12: value 33K -> (none); footprint Resistor_SMD:R_0603_1608Metric_Pad0.98x0.95mm_HandSolder -> (none); LCSC # (none) -> C4216
- R14: value 4K -> (none); footprint Resistor_SMD:R_0603_1608Metric_Pad0.98x0.95mm_HandSolder -> (none); LCSC # (none) -> C23186
- R15: value 100 -> (none); footprint Resistor_SMD:R_0603_1608Metric_Pad0.98x0.95mm_HandSolder -> (none); LCSC # (none) -> C22775
- R16: value 33K -> (none); footprint Resistor_SMD:R_0603_1608Metric_Pad0.98x0.95mm_HandSolder -> (none); 100+ €0.0011 -> (none); 1000+ €0.001 -> (none); LCSC # (none) -> C4216; LCSC Part # C25803 -> (none); LCSC link https://lcsc.com/product-detail/Chip-Resistor-Surface-Mount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 -> (none); Manufacturer UNI-ROYAL(Uniroyal Elec) -> (none); Mfr. Part # 0603WAF1003T5E -> (none); Package 0603 -> (none)
- R17: value 5.1K -> (none); footprint Resistor_SMD:R_0603_1608Metric_Pad0.98x0.95mm_HandSolder -> (none); LCSC # (none) -> C23186
- R2, R3: value 5.1K 1% -> (none); footprint Resistor_SMD:R_0603_1608Metric_Pad0.98x0.95mm_HandSolder -> (none); LCSC # (none) -> C23186; LCSC Part # C23186 -> (none)
- R4, R5: value 220 -> (none); footprint Resistor_SMD:R_0603_1608Metric_Pad0.98x0.95mm_HandSolder -> (none); LCSC # (none) -> C22962; LCSC Part # C22962 -> (none)
- R6, R7: value 10K -> (none); footprint Resistor_SMD:R_0603_1608Metric_Pad0.98x0.95mm_HandSolder -> (none); LCSC # (none) -> C25804; LCSC Part # C25804 -> (none)
- R8, R9: value 100K -> (none); footprint Resistor_SMD:R_0603_1608Metric_Pad0.98x0.95mm_HandSolder -> (none); LCSC # (none) -> C25803
- SW1, SW2, SW3: value TS-1185EC-C-D-B -> (none); footprint footprint:SW-SMD_4P-L3.7-W3.0-P1.50-LS4.7 -> (none)
- U1: value AP40P05 -> (none); footprint footprint:SOT-23-3_L2.9-W1.3-P1.90-LS2.4-BR -> (none)
- U10: value TP4056 -> (none); footprint footprint:ESOP-8_L4.9-W3.9-P1.27-LS6.0-BL-EP -> (none)
- U11: value DW01A -> (none); footprint footprint:SOT-23-6_L2.9-W1.6-P0.95-LS2.8-BL -> (none)
- U18: value BL1117-33CX -> (none); footprint footprint:SOT-223-4_L6.5-W3.5-P2.30-LS7.0-BR -> (none)
- U2, U6: value SS54 -> (none); footprint footprint:SMA_L4.4-W2.8-LS5.4-RD -> (none)
- U20: value MSM261D4030H1CPM -> (none); footprint footprint:MIC-SMD_8P-L3.0-W4.0-P0.85-BL -> (none); LCSC # (none) -> C966942
- U26: value M1250RS-02P -> (none); footprint footprint:CONN-SMD_2P-P1.25_L4.4-W7.4 -> (none)
- U3: LCSC # (none) -> C15741
- U4: value ESP32-WROOM-32E -> (none); footprint footprint:WIFI-SMD_ESP32-WROOM-32E -> (none)
- U5: value FP6298XR-G1 -> (none); footprint footprint:SOP-8_L4.9-W3.9-P1.27-LS6.0-BL-EP -> (none)
- U7: value CP2102-GMR -> (none); footprint footprint:QFN-28_L5.0-W5.0-P0.50-BL-EP -> (none)
- U8: value UMH3N -> (none); footprint footprint:SC-70-6_L2.2-W1.3-P0.65-LS2.1-BR -> (none)
- U9: value FS8205A -> (none); footprint footprint:SOT-23-6_L2.9-W1.6-P0.95-LS2.8-BR -> (none)
- USB1: value U262-161N-4BVC11 -> (none); footprint footprint:USB-3.1-SMD_U262-161N-4BVC11 -> (none)
Other:
- note removed: "Nuts"
- note removed: "PCB connector holes"
- moved on the sheet: C11, C14, C15, D1, D2, R10, R11, R13, R14, R15, R8, R9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

Commit message: added new glowsign design
Parts:
- removed C3: (no value), symbol Device:220uF 10V 6.3x5.4mm
- removed D1: (no value), symbol Device:green_LED_0603
- removed D2: (no value), symbol Device:red LED 0603
- removed D26: (no value), symbol MyParts:WS2812B
- removed R10, R11: (no value), symbol Device:1K_0603
- removed R16: (no value), symbol Device:100K 0603
- removed R17: (no value), symbol Device:R
- removed SW3: (no value), symbol MyParts:TS-1185EC-C-D-B
- removed U1: (no value), symbol MyParts:AP40P05
- removed U5: (no value), symbol MyParts:FP6298XR-G1
- added C22, C23, C29, C30, C31, C52: 0.1uf, Capacitor_SMD:C_0603_1608Metric_Pad1.08x0.95mm_HandSolder, symbol Device:C
- added C3, C55, C56: 220uF, Capacitor_SMD:C_1206_3216Metric_Pad1.33x1.80mm_HandSolder, symbol Device:C
- added D14, D15, D16, D7, D8: WS2812B, LED_SMD:LED_WS2812B_PLCC4_5.0x5.0mm_P3.2mm, symbol MyParts:WS2812B
- added D26, D37: WS2812B-4020, footprint:LED-SMD_WS2812B-4020, symbol MyParts:WS2812B-4020
- added JP1, JP2: SolderJumper_2_Open, Jumper:SolderJumper-2_P1.3mm_Open_RoundedPad1.0x1.5mm, symbol Jumper:SolderJumper_2_Open
- added P1, P2, P3, P4, P5, P6: Thermal_Pad, footprint:Thermal pad, symbol MyParts:Thermal_Pad
- added R10, R11, R16: 100K, Resistor_SMD:R_0603_1608Metric_Pad0.98x0.95mm_HandSolder, symbol Device:R
- added R17: 62K, Resistor_SMD:R_0603_1608Metric_Pad0.98x0.95mm_HandSolder, symbol Device:1K_0603
- added R18, R19, R20, R21: 10K, Resistor_SMD:R_0603_1608Metric_Pad0.98x0.95mm_HandSolder, symbol Device:10K 0603
- added R22: 36K, Resistor_SMD:R_0603_1608Metric_Pad0.98x0.95mm_HandSolder, symbol Device:1K_0603
- added R23: 5.1K, Resistor_SMD:R_0603_1608Metric_Pad0.98x0.95mm_HandSolder, symbol Device:1K_0603
- added SW3: TS24CA, footprint:SW-SMD_TS24CA, symbol MyParts:TS24CA
- added TP1, TP2, TP4, TP5, TP6, TP7, TP8: TestPoint, TestPoint:TestPoint_Pad_D1.5mm, symbol Connector:TestPoint
- added U1: S8050, footprint:SOT-23-3_L3.0-W1.7-P0.95-LS2.9-BR, symbol MyParts:S8050
- added U12: AO3400A, footprint:SOT-23-3_L2.9-W1.6-P1.90-LS2.8-BR, symbol MyParts:AO3400A
- added U13, U14, U16: AP40P05, footprint:SOT-23-3_L2.9-W1.3-P1.90-LS2.4-BR, symbol MyParts:AP40P05
- added U15, U17: SS54, footprint:SMA_L4.4-W2.8-LS5.4-RD, symbol MyParts:SS54
- added U5: FP6276BXR-G1, footprint:SOP-8_L4.9-W3.9-P1.27-LS6.0-BL-EP, symbol MyParts:FP6276BXR-G1
- C1, C11, C14, C5, C7: value (none) -> 10uF; footprint (none) -> Capacitor_SMD:C_0603_1608Metric_Pad1.08x0.95mm_HandSolder
- C10, C15, C2, C6: value (none) -> 0.1uF; footprint (none) -> Capacitor_SMD:C_0603_1608Metric_Pad1.08x0.95mm_HandSolder
- C12, C16: value (none) -> 22uF; footprint (none) -> Capacitor_SMD:C_0603_1608Metric_Pad1.08x0.95mm_HandSolder
- C13: value (none) -> 0.1uf; footprint (none) -> Capacitor_SMD:C_0603_1608Metric_Pad1.08x0.95mm_HandSolder; LCSC # C59461 -> C14663
- C17: value (none) -> 100uF; footprint (none) -> Capacitor_SMD:C_1206_3216Metric_Pad1.33x1.80mm_HandSolder; LCSC # C59461 -> C15008
- C18: renamed from C23; value (none) -> 0.1uf; footprint (none) -> Capacitor_SMD:C_0603_1608Metric_Pad1.08x0.95mm_HandSolder
- C19: renamed from C24; value (none) -> 0.1uf; footprint (none) -> Capacitor_SMD:C_0603_1608Metric_Pad1.08x0.95mm_HandSolder
- C20: renamed from C25; value (none) -> 0.1uf; footprint (none) -> Capacitor_SMD:C_0603_1608Metric_Pad1.08x0.95mm_HandSolder
- C21: renamed from C26; value (none) -> 0.1uf; footprint (none) -> Capacitor_SMD:C_0603_1608Metric_Pad1.08x0.95mm_HandSolder
- C24: renamed from C27; value (none) -> 0.1uf; footprint (none) -> Capacitor_SMD:C_0603_1608Metric_Pad1.08x0.95mm_HandSolder
- C25: renamed from C28; value (none) -> 0.1uf; footprint (none) -> Capacitor_SMD:C_0603_1608Metric_Pad1.08x0.95mm_HandSolder
- C26: renamed from C29; value (none) -> 0.1uf; footprint (none) -> Capacitor_SMD:C_0603_1608Metric_Pad1.08x0.95mm_HandSolder
- C27: renamed from C30; value (none) -> 0.1uf; footprint (none) -> Capacitor_SMD:C_0603_1608Metric_Pad1.08x0.95mm_HandSolder
- C28: renamed from C31; value (none) -> 0.1uf; footprint (none) -> Capacitor_SMD:C_0603_1608Metric_Pad1.08x0.95mm_HandSolder
- C32, C33, C34, C35, C36, C37, C38, C39, C40, C41, C42, C43, C44, C45, C46: value (none) -> 0.1uf; footprint (none) -> Capacitor_SMD:C_0603_1608Metric_Pad1.08x0.95mm_HandSolder
- C4: value (none) -> 4.7uF 6.3V 10%; footprint (none) -> Capacitor_SMD:C_0603_1608Metric_Pad1.08x0.95mm_HandSolder
- C47: renamed from C18; value (none) -> 0.1uf; footprint (none) -> Capacitor_SMD:C_0603_1608Metric_Pad1.08x0.95mm_HandSolder
- C48: renamed from C19; value (none) -> 0.1uf; footprint (none) -> Capacitor_SMD:C_0603_1608Metric_Pad1.08x0.95mm_HandSolder
- C49: renamed from C20; value (none) -> 0.1uf; footprint (none) -> Capacitor_SMD:C_0603_1608Metric_Pad1.08x0.95mm_HandSolder
- C50: renamed from C21; value (none) -> 0.1uf; footprint (none) -> Capacitor_SMD:C_0603_1608Metric_Pad1.08x0.95mm_HandSolder
- C51: renamed from C22; value (none) -> 0.1uf; footprint (none) -> Capacitor_SMD:C_0603_1608Metric_Pad1.08x0.95mm_HandSolder
- C53: renamed from C47; value (none) -> 10uF; footprint (none) -> Capacitor_SMD:C_0603_1608Metric_Pad1.08x0.95mm_HandSolder
- C54: renamed from C48; value (none) -> 0.1uF; footprint (none) -> Capacitor_SMD:C_0603_1608Metric_Pad1.08x0.95mm_HandSolder
- C8, C9: value (none) -> 1uF; footprint (none) -> Capacitor_SMD:C_0603_1608Metric_Pad1.08x0.95mm_HandSolder
- D10: renamed from D13; value (none) -> WS2812B; footprint (none) -> LED_SMD:LED_WS2812B_PLCC4_5.0x5.0mm_P3.2mm
- D11: renamed from D14; value (none) -> WS2812B; footprint (none) -> LED_SMD:LED_WS2812B_PLCC4_5.0x5.0mm_P3.2mm
- D12: renamed from D15; value (none) -> WS2812B; footprint (none) -> LED_SMD:LED_WS2812B_PLCC4_5.0x5.0mm_P3.2mm
- D13: renamed from D16; value (none) -> WS2812B; footprint (none) -> LED_SMD:LED_WS2812B_PLCC4_5.0x5.0mm_P3.2mm
- D17, D18, D19, D20, D21, D22, D23, D24, D25: value (none) -> WS2812B; footprint (none) -> LED_SMD:LED_WS2812B_PLCC4_5.0x5.0mm_P3.2mm
- D27, D28, D29, D30, D31: value (none) -> WS2812B-4020; footprint (none) -> footprint:LED-SMD_WS2812B-4020
- D3: renamed from D8; value (none) -> WS2812B; footprint (none) -> LED_SMD:LED_WS2812B_PLCC4_5.0x5.0mm_P3.2mm
- D32: renamed from D3; value (none) -> WS2812B-4020; footprint (none) -> footprint:LED-SMD_WS2812B-4020
- D33: renamed from D4; value (none) -> WS2812B-4020; footprint (none) -> footprint:LED-SMD_WS2812B-4020
- D34: renamed from D5; value (none) -> WS2812B-4020; footprint (none) -> footprint:LED-SMD_WS2812B-4020
- D35: renamed from D6; value (none) -> WS2812B-4020; footprint (none) -> footprint:LED-SMD_WS2812B-4020
- D36: renamed from D7; value (none) -> WS2812B-4020; footprint (none) -> footprint:LED-SMD_WS2812B-4020
- D4: renamed from D9; value (none) -> WS2812B; footprint (none) -> LED_SMD:LED_WS2812B_PLCC4_5.0x5.0mm_P3.2mm
- D5: renamed from D10; value (none) -> WS2812B; footprint (none) -> LED_SMD:LED_WS2812B_PLCC4_5.0x5.0mm_P3.2mm
- D6: renamed from D11; value (none) -> WS2812B; footprint (none) -> LED_SMD:LED_WS2812B_PLCC4_5.0x5.0mm_P3.2mm
- D9: renamed from D12; value (none) -> WS2812B; footprint (none) -> LED_SMD:LED_WS2812B_PLCC4_5.0x5.0mm_P3.2mm
- F1, F2: value (none) -> BSMD1812-300-16V; footprint (none) -> Fuse:Fuse_1812_4532Metric_Pad1.30x3.40mm_HandSolder
- L1: value (none) -> CKCS5040-3_3UH_M; footprint (none) -> footprint:IND-SMD_L5.0-W5.0
- R1: value (none) -> 62; footprint (none) -> Resistor_SMD:R_0603_1608Metric_Pad0.98x0.95mm_HandSolder
- R12: value (none) -> 100K; footprint (none) -> Resistor_SMD:R_0603_1608Metric_Pad0.98x0.95mm_HandSolder; LCSC # C4216 -> C25803
- R13: value (none) -> 1K; footprint (none) -> Resistor_SMD:R_0603_1608Metric_Pad0.98x0.95mm_HandSolder
- R14, R2, R3: value (none) -> 5.1K; footprint (none) -> Resistor_SMD:R_0603_1608Metric_Pad0.98x0.95mm_HandSolder
- R15: value (none) -> 100; footprint (none) -> Resistor_SMD:R_0603_1608Metric_Pad0.98x0.95mm_HandSolder
- R4, R5: value (none) -> 220; footprint (none) -> Resistor_SMD:R_0603_1608Metric_Pad0.98x0.95mm_HandSolder
- R6, R7: value (none) -> 10K; footprint (none) -> Resistor_SMD:R_0603_1608Metric_Pad0.98x0.95mm_HandSolder
- R8, R9: value (none) -> 100K; footprint (none) -> Resistor_SMD:R_0603_1608Metric_Pad0.98x0.95mm_HandSolder
- SW1, SW2: value (none) -> TS-1185EC-C-D-B; footprint (none) -> footprint:SW-SMD_4P-L3.7-W3.0-P1.50-LS4.7
- U10: value (none) -> TP4056; footprint (none) -> footprint:ESOP-8_L4.9-W3.9-P1.27-LS6.0-BL-EP
- U11: value (none) -> DW01A; footprint (none) -> footprint:SOT-23-6_L2.9-W1.6-P0.95-LS2.8-BL
- U18: value (none) -> BL1117-33CX; footprint (none) -> footprint:SOT-223-4_L6.5-W3.5-P2.30-LS7.0-BR
- U2, U6: value (none) -> SS54; footprint (none) -> footprint:SMA_L4.4-W2.8-LS5.4-RD
- U20: value (none) -> MSM261D4030H1CPM; footprint (none) -> footprint:MIC-SMD_8P-L3.0-W4.0-P0.85-BL
- U26: value (none) -> M1250RS-02P; footprint (none) -> footprint:CONN-SMD_2P-P1.25_L4.4-W7.4
- U3: value (none) -> SN74LVC2T45DCUR; footprint (none) -> footprint:VSSOP-8_L2.4-W2.1-P0.50-LS3.2-BR
- U4: value (none) -> ESP32-WROOM-32E; footprint (none) -> footprint:WIFI-SMD_ESP32-WROOM-32E
- U7: value (none) -> CP2102-GMR; footprint (none) -> footprint:QFN-28_L5.0-W5.0-P0.50-BL-EP
- U8: value (none) -> UMH3N; footprint (none) -> footprint:SC-70-6_L2.2-W1.3-P0.65-LS2.1-BR
- U9: value (none) -> FS8205A; footprint (none) -> footprint:SOT-23-6_L2.9-W1.6-P0.95-LS2.8-BR
- USB1: value (none) -> U262-161N-4BVC11; footprint (none) -> footprint:USB-3.1-SMD_U262-161N-4BVC11
Connections:
- net +3V3: now also TP6.1
- net +5V: now also U2.1 (K), C3.1, C55.1, C56.1, JP1.1 (A), JP2.1 (A), R18.2, R20.2, R21.2, TP8.1, U13.2 (S), U14.2 (S), U15.1 (K), U16.2 (S), U17.1 (K); no longer C16.1, C17.1, C18.1, C19.1, C20.1, C21.1, C24.1, C25.1, C26.1, C27.1, C28.1, C32.1, C33.1, C34.1, C35.1, C36.1, C37.1, C38.1, C39.1, C40.1, C41.1, C42.1, C43.1, C44.1, C45.1, C46.1, C47.1, C48.1, C49.1, C50.1, C51.1, D10.1 (VDD), D11.1 (VDD), D12.1 (VDD), D13.1 (VDD), D17.1 (VDD), D18.1 (VDD), D19.1 (VDD), D20.1 (VDD), D21.1 (VDD), D22.1 (VDD), D23.1 (VDD), D24.1 (VDD), D25.1 (VDD), D27.2 (VDD), D28.2 (VDD), D29.2 (VDD), D3.1 (VDD), D30.2 (VDD), D31.2 (VDD), D32.2 (VDD), D33.2 (VDD), D34.2 (VDD), D35.2 (VDD), D36.2 (VDD), D4.1 (VDD), D5.1 (VDD), D6.1 (VDD), D9.1 (VDD)
- net +BATT: now also TP4.1
- net -BATT: now also TP5.1
- net GND: now also C22.2, C23.2, C29.2, C3.2, C30.2, C31.2, C52.2, C55.2, C56.2, D14.3 (VSS), D15.3 (VSS), D16.3 (VSS), D26.4 (VSS), D37.4 (VSS), D7.3 (VSS), D8.3 (VSS), P1.1, P2.1, P3.1, P4.1, P5.1, P6.1, R11.1, R17.2, R19.1, R23.1, SW3.3, TP7.1, U1.2 (E), U12.2 (S), U5.5 (GND), U5.9 (EP); no longer R12.1
- net IO16/LED1: now also TP1.1
- net LED1 DATA OUT: now also D3.4 (DIN); no longer D32.1 (DIN)
- net at D13.2 (DOUT): now also D14.4 (DIN); no longer D17.4 (DIN)
- net at F2.2: now also C12.1, L1.1, R16.1, U5.3 (VIN)
- net at D31.3 (DOUT): now also D32.1 (DIN)
- net at R12.2: now also U1.1 (B)
- net at U6.2 (A): now also C16.1, C17.1, R22.2, U15.2 (A), U5.8 (VO); no longer L1.2
- net at D27.1 (DIN): now also D26.3 (DOUT)
- net at D36.3 (DOUT): now also D37.1 (DIN); no longer D3.4 (DIN)
- net at D9.4 (DIN): now also D8.2 (DOUT); no longer D6.2 (DOUT)
- net at D25.2 (DOUT): now also D26.1 (DIN)
- net IO27/BATT CHARGING: now reaches U10.7 (CHRG#)
- net IO27/BATT CHARGING: now also U4.12 (IO27)
- net IO25/VBUS: now reaches U4.10 (IO25)
- net IO25/VBUS: now also R10.1, R11.2
- net IO26/BATT VOLT: now reaches U4.11 (IO26)
- net IO26/BATT VOLT: now also R8.1, R9.2
- net IO18/MAINBUTTON: now reaches U4.30 (IO18)
- net IO18/MAINBUTTON: now also SW3.4, TP2.1
- net IO19: now reaches U4.31 (IO19)
- net IO23/LEDPOWER: now reaches U4.37 (IO23)
- net IO23/LEDPOWER: now also R19.2, U12.1 (G)
- removed net I34/BATTVOLT: R8.1, R9.2, U4.6 (I34)
- net IO33/MAINBUTTON: no longer names the net of U4.9 (IO33)
- net RESET renamed EN
- net USB-C 5V renamed VBUS
- net VBUS: now also R12.1, R10.2; no longer F1.2, U2.2 (A)
- new net: D14.2 (DOUT), D15.4 (DIN)
- new net: C13.1, R16.2, U1.3 (C), U5.4 (EN)
- new net: F1.2, U17.2 (A), U2.2 (A)
- new net: R18.1, R20.1, R21.1, U12.3 (D), U13.1 (G), U14.1 (G), U16.1 (G)
- new net: R22.1, R23.2, U5.6 (FB)
- new net: L1.2, U5.1 (LX), U5.2 (LX)
- new net: R17.1, U5.7 (OC)
- new net: D16.2 (DOUT), D17.4 (DIN)
- new net: D15.2 (DOUT), D16.4 (DIN)
- new net: D7.2 (DOUT), D8.4 (DIN)
- new net: D6.2 (DOUT), D7.4 (DIN)
- new net LED 5V: C18.1, C19.1, C20.1, C21.1, C22.1, C23.1, C24.1, C25.1, C26.1, C27.1, C28.1, C29.1, C30.1, C31.1, C32.1, C33.1, C34.1, C35.1, C36.1, C37.1, C38.1, C39.1, C40.1, C41.1, C42.1, C43.1, C44.1, C45.1, C46.1, C47.1, C48.1, C49.1, C50.1, C51.1, C52.1, D10.1 (VDD), D11.1 (VDD), D12.1 (VDD), D13.1 (VDD), D14.1 (VDD), D15.1 (VDD), D16.1 (VDD), D17.1 (VDD), D18.1 (VDD), D19.1 (VDD), D20.1 (VDD), D21.1 (VDD), D22.1 (VDD), D23.1 (VDD), D24.1 (VDD), D25.1 (VDD), D26.2 (VDD), D27.2 (VDD), D28.2 (VDD), D29.2 (VDD), D3.1 (VDD), D30.2 (VDD), D31.2 (VDD), D32.2 (VDD), D33.2 (VDD), D34.2 (VDD), D35.2 (VDD), D36.2 (VDD), D37.2 (VDD), D4.1 (VDD), D5.1 (VDD), D6.1 (VDD), D7.1 (VDD), D8.1 (VDD), D9.1 (VDD), JP1.2 (B), JP2.2 (B), U13.3 (D), U14.3 (D), U16.3 (D)
Other:
- note added: "5V converter (for battery version)"
- note added: "Close to PGND"
- note added: "Define max output: (180000/62000)+0,2 -> 3.1A"
- note added: "Define voltage: 0,6*(1+(36000/5100)) -> 4.8V"
- note added: "Lipo charging & protection (for battery version)"
- note added: "Pins IN/OUT"
- note added: "Thermal Pads"
- note removed: "5V converter"
- note removed: "IOCP = (110.000/R10)+0.3 -> 3.63A current limit"
- note removed: "Lipo charging & protection"
- note removed: "VOUT = 0.6V*(1+R7/R8) -> 5V output voltage"
- moved on the sheet: C18, C19, C2, C20, C21, C24, C25, C26, C27, C28, C47, C48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
