File: Main PCB/GlowSignMainPCB.kicad_sch (KiCad schematic)
At the start: 156 parts, among them P1 Thermal_Pad, P2 Thermal_Pad, P3 Thermal_Pad, P4 Thermal_Pad, P5 Thermal_Pad, P6 Thermal_Pad, SW1 TS-1185EC-C-D-B, SW2 TS-1185EC-C-D-B, SW3 TS24CA, U1 S8050, U10 TP4056, U11 DW01A, U12 AO3400A, U13 AP40P05, U14 AP40P05, U15 SS54, U16 AP40P05, U17 SS54, U18 BL1117-33CX, U2 SS54, U20 MSM261D4030H1CPM, U26 M1250RS-02P, U3 SN74LVC2T45DCUR, U4 ESP32-WROOM-32E, U5 FP6276BXR-G1, U6 SS54, U7 CP2102-GMR, U8 UMH3N, U9 FS8205A

Commit message: fixed important mistake... VBUS not connected...
Parts:
- removed P1, P2, P3, P4, P5, P6: Thermal_Pad, footprint:Thermal pad, symbol MyParts:Thermal_Pad
Connections:
- net VBUS: now also F1.2, U17.2 (A), U2.2 (A)
Other:
- note removed: "Thermal Pads"
