File: Main PCB/GlowSignMainPCB.kicad_sch (KiCad schematic)
At the start: 150 parts, among them SW1 TS-1185EC-C-D-B, SW2 TS-1185EC-C-D-B, SW3 TS24CA, U1 S8050, U10 TP4056, U11 DW01A, U12 AO3400A, U13 AP40P05, U14 AP40P05, U15 SS54, U16 AP40P05, U17 SS54, U18 BL1117-33CX, U2 SS54, U20 MSM261D4030H1CPM, U26 M1250RS-02P, U3 SN74LVC2T45DCUR, U4 ESP32-WROOM-32E, U5 FP6276BXR-G1, U6 SS54, U7 CP2102-GMR, U8 UMH3N, U9 FS8205A

Commit message: separated battery electronics into separate pcb
Parts:
- removed C11, C14: 10uF, Capacitor_SMD:C_0603_1608Metric_Pad1.08x0.95mm_HandSolder, symbol Device:10uF 0603
- removed C12, C16: 22uF, Capacitor_SMD:C_0603_1608Metric_Pad1.08x0.95mm_HandSolder, symbol Device:C
- removed C13: 0.1uf, Capacitor_SMD:C_0603_1608Metric_Pad1.08x0.95mm_HandSolder, symbol Device:C
- removed C15: 0.1uF, Capacitor_SMD:C_0603_1608Metric_Pad1.08x0.95mm_HandSolder, symbol Device:0.1uF_0603
- removed C17: 100uF, Capacitor_SMD:C_1206_3216Metric_Pad1.33x1.80mm_HandSolder, symbol Device:C
- removed F2: BSMD1812-300-16V, Fuse:Fuse_1812_4532Metric_Pad1.30x3.40mm_HandSolder, symbol Device:Fuse
- removed L1: CKCS5040-3_3UH_M, footprint:IND-SMD_L5.0-W5.0, symbol MyParts:CKCS5040-3_3UH_M
- removed R12, R16, R8, R9: 100K, Resistor_SMD:R_0603_1608Metric_Pad0.98x0.95mm_HandSolder, symbol Device:R
- removed R13: 1K, Resistor_SMD:R_0603_1608Metric_Pad0.98x0.95mm_HandSolder, symbol Device:1K_0603
- removed R14: 5.1K, Resistor_SMD:R_0603_1608Metric_Pad0.98x0.95mm_HandSolder, symbol Device:R
- removed R15: 100, Resistor_SMD:R_0603_1608Metric_Pad0.98x0.95mm_HandSolder, symbol Device:R
- removed R17: 62K, Resistor_SMD:R_0603_1608Metric_Pad0.98x0.95mm_HandSolder, symbol Device:1K_0603
- removed R22: 36K, Resistor_SMD:R_0603_1608Metric_Pad0.98x0.95mm_HandSolder, symbol Device:1K_0603
- removed R23: 5.1K, Resistor_SMD:R_0603_1608Metric_Pad0.98x0.95mm_HandSolder, symbol Device:1K_0603
- removed U1: S8050, footprint:SOT-23-3_L3.0-W1.7-P0.95-LS2.9-BR, symbol MyParts:S8050
- removed U10: TP4056, footprint:ESOP-8_L4.9-W3.9-P1.27-LS6.0-BL-EP, symbol MyParts:TP4056
- removed U11: DW01A, footprint:SOT-23-6_L2.9-W1.6-P0.95-LS2.8-BL, symbol MyParts:DW01A
- removed U15, U6: SS54, footprint:SMA_L4.4-W2.8-LS5.4-RD, symbol MyParts:SS54
- removed U26: M1250RS-02P, footprint:CONN-SMD_2P-P1.25_L4.4-W7.4, symbol MyParts:M1250RS-02P
- removed U5: FP6276BXR-G1, footprint:SOP-8_L4.9-W3.9-P1.27-LS6.0-BL-EP, symbol MyParts:FP6276BXR-G1
- removed U9: FS8205A, footprint:SOT-23-6_L2.9-W1.6-P0.95-LS2.8-BR, symbol MyParts:FS8205A
- added C57: 0.1uF, Capacitor_SMD:C_0603_1608Metric_Pad1.08x0.95mm_HandSolder, symbol Device:0.1uF 0603
- added P1, P2: Solder_Pad, footprint:Solder pad, symbol MyParts:Solder_Pad
- added U19: TPS3839G33DBZR, footprint:SOT-23-3_L2.9-W1.3-P1.90-LS2.4-BR, symbol MyParts:TPS3839G33DBZR
Connections:
- net +3V3: now also C57.1, U19.3 (VDD)
- net +BATT: now also P1.1
- net -BATT: now also P2.1
- net EN: now also U19.2 (RESET#)
- net GND: now also C57.2, U19.1 (GND)
Other:
- note removed: "5V converter (for battery version)"
- note removed: "Close to PGND"
- note removed: "Define max output: (180000/62000)+0,2 -> 3.1A"
- note removed: "Define voltage: 0,6*(1+(36000/5100)) -> 4.8V"
- note removed: "Lipo charging & protection (for battery version)"
- note removed: "Programm charging speed with resistor: 10K => 130 mA 5K => 250mA 4K => 300mA 3K => 400mA 2K => 580mA 1.66K => 690mA 1.5K => 780mA 1.33K => 900mA 1.2K => 1000mA"
- moved on the sheet: C5, C7, U18

Commit message: updated pcb files
Parts:
- removed C51, C52: 0.1uf, Capacitor_SMD:C_0603_1608Metric_Pad1.08x0.95mm_HandSolder, symbol Device:C
- removed D26, D27, D28, D29, D30, D31, D32, D33, D34, D35, D36, D37: WS2812B-4020, footprint:LED-SMD_WS2812B-4020, symbol MyParts:WS2812B-4020
- added D26, D27, D28, D29, D30, D31, D32, D33, D34, D35: WS2812B, LED_SMD:LED_WS2812B_PLCC4_5.0x5.0mm_P3.2mm, symbol MyParts:WS2812B
- added JP3: SolderJumper_2_Bridged, Jumper:SolderJumper-2_P1.3mm_Bridged_RoundedPad1.0x1.5mm, symbol Jumper:SolderJumper_2_Bridged
- added P3, P4, P5, P6, P7: Solder_Pad, footprint:Solder pad, symbol MyParts:Solder_Pad
Connections:
- net +3V3: now also JP3.1 (A); no longer C10.2, C53.2, U20.1 (VDD)
- net +5V: now also P6.1
- net GND: now also D26.3 (VSS), D27.3 (VSS), D28.3 (VSS), D29.3 (VSS), D30.3 (VSS), D31.3 (VSS), D32.3 (VSS), D33.3 (VSS), D34.3 (VSS), D35.3 (VSS), P7.1
- net IO26/BATT VOLT: now also P3.1
- net IO27/BATT CHARGING: now also P5.1
- net LED 5V: now also D26.1 (VDD), D27.1 (VDD), D28.1 (VDD), D29.1 (VDD), D30.1 (VDD), D31.1 (VDD), D32.1 (VDD), D33.1 (VDD), D34.1 (VDD), D35.1 (VDD)
- net VBUS: now also P4.1
- net at D25.2 (DOUT): now also D26.4 (DIN)
- new net: D33.2 (DOUT), D34.4 (DIN)
- new net: D32.2 (DOUT), D33.4 (DIN)
- new net: D31.2 (DOUT), D32.4 (DIN)
- new net: D30.2 (DOUT), D31.4 (DIN)
- new net: C10.2, C53.2, JP3.2 (B), U20.1 (VDD)
- new net: D27.2 (DOUT), D28.4 (DIN)
- new net: D26.2 (DOUT), D27.4 (DIN)
- new net: D34.2 (DOUT), D35.4 (DIN)
- new net: D29.2 (DOUT), D30.4 (DIN)
- new net: D28.2 (DOUT), D29.4 (DIN)
Other:
- note added: "Battery Extension"
- moved on the sheet: C41, C42, C43, C44, C45, C46, C47, C48, C49, C50, P1, P2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

Commit message: replaced 0603 with 0402 (battery extension)
Connections:
- net IO18/MAINBUTTON: no longer SW3.4, U4.30 (IO18)
- net IO33/MAINBUTTON: now reaches U4.9 (IO33)
- net IO33/MAINBUTTON: now also SW3.4
Changed lines of the file:
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@@
-    (stroke (width 0) (type default) (color 0 0 0 0))
-  )
-  (wire (pts (xy 81.28 74.93) (xy 83.82 74.93))
     (stroke (width 0) (type default) (color 0 0 0 0))
   )
@@
   )
   (wire (pts (xy 172.72 312.42) (xy 176.53 312.42))
+    (stroke (width 0) (type default) (color 0 0 0 0))
+  )
+  (wire (pts (xy 81.28 97.79) (xy 83.82 97.79))
     (stroke (width 0) (type default) (color 0 0 0 0))
   )
@@
     )
   )
-  (global_label "IO18{slash}MAINBUTTON" (shape input) (at 83.82 74.93 0) (fields_autoplaced)
-    (effects (font (size 1.27 1.27)) (justify left))
-    (property "Intersheet References" "${INTERSHEET_REFS}" (id 0) (at 103.5898 74.8506 0)
+  (global_label "IO33{slash}MAINBUTTON" (shape input) (at 83.82 97.79 0) (fields_autoplaced)
+    (effects (font (size 1.27 1.27)) (justify left))
+    (property "Intersheet References" "${INTERSHEET_REFS}" (id 0) (at 103.5898 97.7106 0)
       (effects (font (size 1.27 1.27)) (justify left) hide)
     )
@@
     )
   )
-  (global_label "IO18{slash}MAINBUTTON" (shape input) (at 547.37 158.75 0) (fields_autoplaced)
+  (global_label "IO33{slash}MAINBUTTON" (shape input) (at 547.37 158.75 0) (fields_autoplaced)
     (effects (font (size 1.27 1.27)) (justify left))
     (property "Intersheet References" "${INTERSHEET_REFS}" (id 0) (at 567.1398 158.6706 0)

Commit message: updated pcb designs
Parts:
- removed C56: 220uF, Capacitor_SMD:C_1206_3216Metric_Pad1.33x1.80mm_HandSolder, symbol Device:C
- removed JP1, JP2: SolderJumper_2_Open, Jumper:SolderJumper-2_P1.3mm_Open_RoundedPad1.0x1.5mm, symbol Jumper:SolderJumper_2_Open
- removed R21: 10K, Resistor_SMD:R_0603_1608Metric_Pad0.98x0.95mm_HandSolder, symbol Device:10K 0603
- removed U16: AP40P05, footprint:SOT-23-3_L2.9-W1.3-P1.90-LS2.4-BR, symbol MyParts:AP40P05
- removed U17: SS54, footprint:SMA_L4.4-W2.8-LS5.4-RD, symbol MyParts:SS54
- R11: value 100K -> 160K; LCSC # C25803 -> C22813
Connections:
- net IO18/MAINBUTTON is gone; now on net IO33/MAINBUTTON: TP2.1
- net +3V3: now also R20.2, U14.2 (S); no longer C2.1, JP3.1 (A), TP6.1, U3.8 (VCCB)
- net +5V: no longer C3.1, C54.1, C55.1, R20.2, U14.2 (S), U3.1 (VCCA)
- net LED 5V: now also C3.1, C54.1, C55.1, U3.1 (VCCA); no longer U14.3 (D)
- new net 3.3V AFTER RELAY: C2.1, JP3.1 (A), TP6.1, U14.3 (D), U3.8 (VCCB)
Other:
- note added: "To Do: fix CP2102 power consumption in sleep mode"
- note added: "To Do: fix constant on/off switching"
- moved on the sheet: C3, C55, F1

Commit message: fixed deep sleep power consumption + new LED0
Parts:
- removed C57: 0.1uF, Capacitor_SMD:C_0603_1608Metric_Pad1.08x0.95mm_HandSolder, symbol Device:0.1uF 0603
- removed U19: TPS3839G33DBZR, footprint:SOT-23-3_L2.9-W1.3-P1.90-LS2.4-BR, symbol MyParts:TPS3839G33DBZR
- added R8, R9: 10K, Resistor_SMD:R_0603_1608Metric_Pad0.98x0.95mm_HandSolder, symbol Device:10K 0603
- added U1: AP40P05, footprint:SOT-23-3_L2.9-W1.3-P1.90-LS2.4-BR, symbol MyParts:AP40P05
- added U5: AO3400A, footprint:SOT-23-3_L2.9-W1.6-P1.90-LS2.8-BR, symbol MyParts:AO3400A
- C8: value 1uF -> 10uF; LCSC # C15849 -> C19702
Connections:
- net +3V3: now also R8.2, U1.2 (S); no longer C4.2, C6.1, U7.6 (VDD), U7.7 (REGIN)
- net +BATT: no longer TP4.1
- net -BATT: no longer TP5.1
- net EN: now also C8.2; no longer C8.1
- net GND: now also C8.1, R9.1, U5.2 (S); no longer C8.2
- net IO16/LED1: no longer TP1.1
- net IO33/MAINBUTTON: no longer TP2.1
- net VBUS: now also R9.2, U5.1 (G)
- net IO12/TDI: now reaches U4.14 (IO12)
- net IO12/TDI: now also TP1.1
- net IO13/TCK: now reaches U4.16 (IO13)
- net IO13/TCK: now also TP2.1
- net 3.3V AFTER RELAY renamed 3.3V AFTER MOSFET
- net IO14/SCK renamed IO14/SCK/TMS
- net IO14/SCK/TMS: now also TP4.1
- net IO15/WS renamed IO15/WS/TDO
- net IO15/WS/TDO: now also TP5.1
- net IO23/LEDPOWER renamed IO23/POWERMOSFETS
- net LED 5V renamed 5V AFTER MOSFET
- new net: C4.2, C6.1, U1.3 (D), U7.6 (VDD), U7.7 (REGIN)
- new net: R8.1, U1.1 (G), U5.3 (D)
Other:
- note added: "Pins 12,13,14,15 for JTAG debugger"
- note removed: "To Do: fix CP2102 power consumption in sleep mode"
- note removed: "To Do: fix constant on/off switching"
- moved on the sheet: C10, C18, C19, C20, C21, C22, C23, C24, C25, C26, C27, C28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

Commit message: updated case design
Parts:
- added SW4: TS24CA, footprint:SW-SMD_TS24CA, symbol MyParts:TS24CA
- added U6: SN74LVC1G373DBVR, footprint:SOT-23-6_L2.9-W1.6-P0.95-LS2.8-BR, symbol MyParts:SN74LVC1G373DBVR
Connections:
- net +3V3: now also SW3.3, SW4.3, U6.5 (VCC)
- net GND: now also U6.2 (GND); no longer SW3.3
- net IO23/POWERMOSFETS: now also U6.3 (D); no longer R19.2, U12.1 (G)
- net IO4/BUTTON 2: now reaches U4.26 (IO4)
- net IO4/BUTTON 2: now also SW4.4
- net IO22/LED LETCH EN: now reaches U4.36 (IO22)
- net IO22/LED LETCH EN: now also U6.1 (LE)
- net IO19: no longer names the net of U4.31 (IO19)
- new net: R19.2, U12.1 (G), U6.4 (Q)
Other:
- note removed: "Keep pressed to start/end deep sleep, press once to cycle animations, press twice or three times to switch to specific animation."
- moved on the sheet: C3, C55, R18, R19, R20, U12, U13, U14
